Commit message: Add differential drive wheels, centralize colors and parameters

File: toy_robot_ws/src/toy_robot_description/urdf/arm_6dof.xacro (robot description, xacro)
@@ -14,6 +14,6 @@
             </geometry>
             <origin xyz="0 0 ${shoulder_length/2}" rpy="0 0 0" />
-            <material name="blue">
-                <color rgba="0 0 0.5 1" />
+            <material name="arm_joint">
+                <color rgba="${color_joint}" />
             </material>
         </visual>
@@ -43,6 +43,6 @@
             </geometry>
             <origin xyz="0 0 ${arm_length/2}" rpy="0 0 0" />
-            <material name="gray">
-                <color rgba="0.5 0.5 0.5 1" />
+            <material name="arm_link1">
+                <color rgba="${color_link}" />
             </material>
         </visual>
@@ -72,6 +72,6 @@
             </geometry>
             <origin xyz="0 0 ${elbow_length/2}" rpy="0 0 0" />
-            <material name="blue">
-                <color rgba="0 0 0.5 1" />
+            <material name="arm_joint2">
+                <color rgba="${color_joint}" />
             </material>
         </visual>
@@ -101,6 +101,6 @@
             </geometry>
             <origin xyz="0 0 ${forearm_length/2}" rpy="0 0 0" />
-            <material name="gray">
-                <color rgba="0.5 0.5 0.5 1" />
+            <material name="arm_link2">
+                <color rgba="${color_link}" />
             </material>
         </visual>
@@ -130,6 +130,6 @@
             </geometry>
             <origin xyz="0 0 ${wrist_height/2}" rpy="0 0 0" />
-            <material name="blue">
-                <color rgba="0 0 0.5 1" />
+            <material name="arm_joint3">
+                <color rgba="${color_joint}" />
             </material>
         </visual>
@@ -158,6 +158,6 @@
             </geometry>
             <origin xyz="0 0 ${hand_height/2}" rpy="0 0 0" />
-            <material name="gray">
-                <color rgba="0.5 0.5 0.5 1" />
+            <material name="arm_link3">
+                <color rgba="${color_link}" />
             </material>
         </visual>

File: toy_robot_ws/src/toy_robot_description/urdf/base_mobile.xacro (robot description, xacro)
@@ -5,5 +5,5 @@
         <parent link="base_footprint" />
         <child link="base_link" />
-        <origin xyz="0 0 0.01" rpy="0 0 0" />
+        <origin xyz="0 0 ${wheel_radius}" rpy="0 0 0" />
     </joint>
     <link name="base_link">

File: toy_robot_ws/src/toy_robot_description/urdf/camera.xacro (robot description, xacro)
@@ -12,6 +12,6 @@
                 <box size="${camera_size_x} ${camera_size_y} ${camera_size_z}" />
             </geometry>
-            <material name="camera_black">
-                <color rgba="0.12 0.12 0.12 1.0" />
+            <material name="camera_body">
+                <color rgba="${color_camera}" />
             </material>
         </visual>

File: toy_robot_ws/src/toy_robot_description/urdf/dimensions.xacro (robot description, xacro)
@@ -42,3 +42,20 @@
     <xacro:property name="finger_y_offset" value="0.02" />
     <xacro:property name="finger_open_max" value="0.025" />
+    <!-- Wheels -->
+    <xacro:property name="wheel_radius" value="0.05" />
+    <xacro:property name="wheel_width" value="0.03" />
+    <xacro:property name="wheel_mass" value="0.1" />
+    <xacro:property name="caster_radius" value="0.02" />
+    <xacro:property name="caster_mass" value="0.05" />
+    <!-- wheel axle Y: just outside the base cylinder -->
+    <xacro:property name="wheel_y" value="${base_radius + wheel_width/2}" />
+    <!-- Colors (RGBA) -->
+    <!-- joints: dark steel -->
+    <xacro:property name="color_joint" value="0.45 0.45 0.48 1.0" />
+    <!-- links: light gray -->
+    <xacro:property name="color_link" value="0.65 0.65 0.65 1.0" />
+    <!-- camera: near white -->
+    <xacro:property name="color_camera" value="0.88 0.88 0.88 1.0" />
+    <!-- rubber dark -->
+    <xacro:property name="color_wheel" value="0.15 0.15 0.15 1.0" />
 </robot>

File: toy_robot_ws/src/toy_robot_description/urdf/toy_robot.urdf.xacro (robot description, xacro)
@@ -3,4 +3,5 @@
     <xacro:include filename="$(find toy_robot_description)/urdf/dimensions.xacro" />
     <xacro:include filename="$(find toy_robot_description)/urdf/base_mobile.xacro" />
+    <xacro:include filename="$(find toy_robot_description)/urdf/wheels.xacro" />
     <xacro:include filename="$(find toy_robot_description)/urdf/camera.xacro" />
     <xacro:include filename="$(find toy_robot_description)/urdf/arm_6dof.xacro" />

Commit message: fix(urdf): parametrize all inertia values and hard-coded box geometry

File: toy_robot_ws/src/toy_robot_description/urdf/arm_6dof.xacro (robot description, xacro)
@@ -27,5 +27,10 @@
             <origin xyz="0 0 ${shoulder_length/2}" rpy="0 0 0" />
             <mass value="${shoulder_mass}" />
-            <inertia ixx="0.000037" ixy="0.0" ixz="0.0" iyy="0.000037" iyz="0.0" izz="0.000024" />
+            <inertia
+                ixx="${shoulder_mass * (3 * shoulder_radius * shoulder_radius + shoulder_length * shoulder_length) / 12}"
+                ixy="0.0" ixz="0.0"
+                iyy="${shoulder_mass * (3 * shoulder_radius * shoulder_radius + shoulder_length * shoulder_length) / 12}"
+                iyz="0.0"
+                izz="${shoulder_mass * shoulder_radius * shoulder_radius / 2}" />
         </inertial>
     </link>
@@ -56,5 +61,10 @@
             <origin xyz="0 0 ${arm_length/2}" rpy="0 0 0" />
             <mass value="${arm_mass}" />
-            <inertia ixx="0.000296" ixy="0.0" ixz="0.0" iyy="0.000296" iyz="0.0" izz="0.000020" />
+            <inertia
+                ixx="${arm_mass * (3 * arm_radius * arm_radius + arm_length * arm_length) / 12}"
+                ixy="0.0" ixz="0.0"
+                iyy="${arm_mass * (3 * arm_radius * arm_radius + arm_length * arm_length) / 12}"
+                iyz="0.0"
+                izz="${arm_mass * arm_radius * arm_radius / 2}" />
         </inertial>
     </link>
@@ -85,5 +95,10 @@
             <origin xyz="0 0 ${elbow_length/2}" rpy="0 0 0" />
             <mass value="${elbow_mass}" />
-            <inertia ixx="0.000015" ixy="0.0" ixz="0.0" iyy="0.000015" iyz="0.0" izz="0.000019" />
+            <inertia
+                ixx="${elbow_mass * (3 * elbow_radius * elbow_radius + elbow_length * elbow_length) / 12}"
+                ixy="0.0" ixz="0.0"
+                iyy="${elbow_mass * (3 * elbow_radius * elbow_radius + elbow_length * elbow_length) / 12}"
+                iyz="0.0"
+                izz="${elbow_mass * elbow_radius * elbow_radius / 2}" />
         </inertial>
     </link>
@@ -114,5 +129,10 @@
             <origin xyz="0 0 ${forearm_length/2}" rpy="0 0 0" />
             <mass value="${forearm_mass}" />
-            <inertia ixx="0.000145" ixy="0.0" ixz="0.0" iyy="0.000145" iyz="0.0" izz="0.000010" />
+            <inertia
+                ixx="${forearm_mass * (3 * forearm_radius * forearm_radius + forearm_length * forearm_length) / 12}"
+                ixy="0.0" ixz="0.0"
+                iyy="${forearm_mass * (3 * forearm_radius * forearm_radius + forearm_length * forearm_length) / 12}"
+                iyz="0.0"
+                izz="${forearm_mass * forearm_radius * forearm_radius / 2}" />
         </inertial>
     </link>
@@ -127,5 +147,5 @@
         <visual>
             <geometry>
-                <box size="0.04 0.04 0.03" />
+                <box size="${wrist_size_x} ${wrist_size_y} ${wrist_height}" />
             </geometry>
             <origin xyz="0 0 ${wrist_height/2}" rpy="0 0 0" />
@@ -136,5 +156,5 @@
         <collision>
             <geometry>
-                <box size="0.04 0.04 0.03" />
+                <box size="${wrist_size_x} ${wrist_size_y} ${wrist_height}" />
             </geometry>
             <origin xyz="0 0 ${wrist_height/2}" rpy="0 0 0" />
@@ -143,5 +163,10 @@
             <origin xyz="0 0 ${wrist_height/2}" rpy="0 0 0" />
             <mass value="${wrist_mass}" />
-            <inertia ixx="0.0000095" ixy="0.0" ixz="0.0" iyy="0.0000095" iyz="0.0" izz="0.000016" />
+            <inertia
+                ixx="${wrist_mass * (wrist_size_y * wrist_size_y + wrist_height * wrist_height) / 12}"
+                ixy="0.0" ixz="0.0"
+                iyy="${wrist_mass * (wrist_size_x * wrist_size_x + wrist_height * wrist_height) / 12}"
+                iyz="0.0"
+                izz="${wrist_mass * (wrist_size_x * wrist_size_x + wrist_size_y * wrist_size_y) / 12}" />
         </inertial>
     </link>
@@ -155,5 +180,5 @@
         <visual>
             <geometry>
-                <box size="0.05 0.05 0.02" />
+                <box size="${hand_size_x} ${hand_size_y} ${hand_height}" />
             </geometry>
             <origin xyz="0 0 ${hand_height/2}" rpy="0 0 0" />
@@ -164,5 +189,5 @@
         <collision>
             <geometry>
-                <box size="0.05 0.05 0.02" />
+                <box size="${hand_size_x} ${hand_size_y} ${hand_height}" />
             </geometry>
             <origin xyz="0 0 ${hand_height/2}" rpy="0 0 0" />
@@ -171,5 +196,10 @@
             <origin xyz="0 0 ${hand_height/2}" rpy="0 0 0" />
             <mass value="${hand_mass}" />
-            <inertia ixx="0.0000208" ixy="0.0" ixz="0.0" iyy="0.0000208" iyz="0.0" izz="0.0000417" />
+            <inertia
+                ixx="${hand_mass * (hand_size_y * hand_size_y + hand_height * hand_height) / 12}"
+                ixy="0.0" ixz="0.0"
+                iyy="${hand_mass * (hand_size_x * hand_size_x + hand_height * hand_height) / 12}"
+                iyz="0.0"
+                izz="${hand_mass * (hand_size_x * hand_size_x + hand_size_y * hand_size_y) / 12}" />
         </inertial>
     </link>

File: toy_robot_ws/src/toy_robot_description/urdf/base_mobile.xacro (robot description, xacro)
@@ -26,5 +26,10 @@
             <origin xyz="0 0 ${base_height/2}" rpy="0 0 0" />
             <mass value="${base_mass}" />
-            <inertia ixx="0.0216666667" ixy="0.0" ixz="0.0" iyy="0.0216666667" iyz="0.0" izz="0.04" />
+            <inertia
+                ixx="${base_mass * (3 * base_radius * base_radius + base_height * base_height) / 12}"
+                ixy="0.0" ixz="0.0"
+                iyy="${base_mass * (3 * base_radius * base_radius + base_height * base_height) / 12}"
+                iyz="0.0"
+                izz="${base_mass * base_radius * base_radius / 2}" />
         </inertial>
     </link>

File: toy_robot_ws/src/toy_robot_description/urdf/camera.xacro (robot description, xacro)
@@ -25,6 +25,10 @@
             <origin xyz="0 0 ${camera_size_z/2}" rpy="0 0 0" />
             <mass value="${camera_mass}" />
-            <inertia ixx="0.0000608333" ixy="0.0" ixz="0.0" iyy="0.0000208333" iyz="0.0"
-                izz="0.0000666667" />
+            <inertia
+                ixx="${camera_mass * (camera_size_y * camera_size_y + camera_size_z * camera_size_z) / 12}"
+                ixy="0.0" ixz="0.0"
+                iyy="${camera_mass * (camera_size_x * camera_size_x + camera_size_z * camera_size_z) / 12}"
+                iyz="0.0"
+                izz="${camera_mass * (camera_size_x * camera_size_x + camera_size_y * camera_size_y) / 12}" />
         </inertial>
     </link>

File: toy_robot_ws/src/toy_robot_description/urdf/dimensions.xacro (robot description, xacro)
@@ -18,5 +18,9 @@
     <xacro:property name="forearm_length" value="0.12" />
     <xacro:property name="wrist_height" value="0.03" />
+    <xacro:property name="wrist_size_x" value="0.04" />
+    <xacro:property name="wrist_size_y" value="0.04" />
     <xacro:property name="hand_height" value="0.02" />
+    <xacro:property name="hand_size_x" value="0.05" />
+    <xacro:property name="hand_size_y" value="0.05" />
     <xacro:property name="shoulder_radius" value="0.020" />
     <xacro:property name="arm_radius" value="0.015" />

File: toy_robot_ws/src/toy_robot_description/urdf/gripper.xacro (robot description, xacro)
@@ -26,5 +26,10 @@
             <origin xyz="0 0 ${palm_z/2}" rpy="0 0 0" />
             <mass value="${palm_mass}" />
-            <inertia ixx="0.0000060" ixy="0.0" ixz="0.0" iyy="0.0000073" iyz="0.0" izz="0.0000137" />
+            <inertia
+                ixx="${palm_mass * (palm_y * palm_y + palm_z * palm_z) / 12}"
+                ixy="0.0" ixz="0.0"
+                iyy="${palm_mass * (palm_x * palm_x + palm_z * palm_z) / 12}"
+                iyz="0.0"
+                izz="${palm_mass * (palm_x * palm_x + palm_y * palm_y) / 12}" />
         </inertial>
     </link>
@@ -56,5 +61,10 @@
             <origin xyz="0 0 ${finger_z/2}" rpy="0 0 0" />
             <mass value="${finger_mass}" />
-            <inertia ixx="0.0000027" ixy="0.0" ixz="0.0" iyy="0.0000026" iyz="0.0" izz="0.0000003" />
+            <inertia
+                ixx="${finger_mass * (finger_y * finger_y + finger_z * finger_z) / 12}"
+                ixy="0.0" ixz="0.0"
+                iyy="${finger_mass * (finger_x * finger_x + finger_z * finger_z) / 12}"
+                iyz="0.0"
+                izz="${finger_mass * (finger_x * finger_x + finger_y * finger_y) / 12}" />
         </inertial>
     </link>
@@ -86,5 +96,10 @@
             <origin xyz="0 0 ${finger_z/2}" rpy="0 0 0" />
             <mass value="${finger_mass}" />
-            <inertia ixx="0.0000027" ixy="0.0" ixz="0.0" iyy="0.0000026" iyz="0.0" izz="0.0000003" />
+            <inertia
+                ixx="${finger_mass * (finger_y * finger_y + finger_z * finger_z) / 12}"
+                ixy="0.0" ixz="0.0"
+                iyy="${finger_mass * (finger_x * finger_x + finger_z * finger_z) / 12}"
+                iyz="0.0"
+                izz="${finger_mass * (finger_x * finger_x + finger_y * finger_y) / 12}" />
         </inertial>
     </link>

Commit message: feat(description): add Gazebo simulation stack with validated robot
- Add gazebo.launch.xml: launches Gazebo, robot_state_publisher, spawner, ros_gz_bridge, RViz
- Add gazebo_plugins.xacro: diff_drive plugin, camera sensor plugin
- Add gz_bridge.yaml: topic mappings for cmd_vel, odom, tf, joint_states, camera
- Add toy_robot_world.sdf: custom world with inline ground plane, light, and gz-sim-sensors-system plugin
- Update CMakeLists.txt: install config, launch, worlds directories
- Update toy_robot.urdf.xacro: include gazebo_plugins.xacro
- Update arm_6dof.xacro, gripper.xacro: minor corrections
- Update package.xml: add ros_gz_sim and ros_gz_bridge exec_depends
- Add docs/simulation_validation_commands.md: full command reference for simulation validation
- Update docs/index.md and README.md: reference new simulation validation guide

Validated: cmd_vel, odom, TF chain, camera image stream, keyboard teleop

File: toy_robot_ws/src/toy_robot_description/urdf/arm_6dof.xacro (robot description, xacro)
@@ -6,4 +6,5 @@
         <origin xyz="${arm_mount_x} 0 ${arm_mount_z}" rpy="0 0 0" />
         <axis xyz="0 0 1" />
+        <dynamics damping="5.0" friction="2.0" />
         <limit effort="1000.0" velocity="1.0" lower="-3.14" upper="3.14" />
     </joint>
@@ -40,4 +41,5 @@
         <origin xyz="0 0 ${shoulder_length}" rpy="0 0 0" />
         <axis xyz="0 1 0" />
+        <dynamics damping="5.0" friction="2.0" />
         <limit effort="1000.0" velocity="1.0" lower="-1.57" upper="1.57" />
     </joint>
@@ -74,4 +76,5 @@
         <origin xyz="0 0 ${arm_length}" rpy="0 0 0" />
         <axis xyz="0 1 0" />
+        <dynamics damping="5.0" friction="2.0" />
         <limit effort="1000.0" velocity="1.0" lower="-1.57" upper="1.57" />
     </joint>
@@ -108,4 +111,5 @@
         <origin xyz="0 0 ${elbow_length}" rpy="0 0 0" />
         <axis xyz="0 0 1" />
+        <dynamics damping="5.0" friction="2.0" />
         <limit effort="1000.0" velocity="1.0" lower="-3.14" upper="3.14" />
     </joint>
@@ -142,4 +146,5 @@
         <origin xyz="0 0 ${forearm_length}" rpy="0 0 0" />
         <axis xyz="0 1 0" />
+        <dynamics damping="5.0" friction="2.0" />
         <limit effort="1000.0" velocity="1.0" lower="-1.57" upper="1.57" />
     </joint>
@@ -176,4 +181,5 @@
         <origin xyz="0 0 ${wrist_height}" rpy="0 0 0" />
         <axis xyz="0 0 1" />
+        <dynamics damping="5.0" friction="2.0" />
     </joint>
     <link name="hand_link">

File: toy_robot_ws/src/toy_robot_description/urdf/gripper.xacro (robot description, xacro)
@@ -40,4 +40,5 @@
         <origin xyz="0 ${finger_y_offset} ${palm_z}" rpy="0 0 0" />
         <axis xyz="0 1 0" />
+        <dynamics damping="10.0" friction="5.0" />
         <limit effort="100.0" velocity="0.5" lower="0.0" upper="${finger_open_max}" />
     </joint>
@@ -75,4 +76,5 @@
         <origin xyz="0 -${finger_y_offset} ${palm_z}" rpy="0 0 0" />
         <axis xyz="0 -1 0" />
+        <dynamics damping="10.0" friction="5.0" />
         <limit effort="100.0" velocity="0.5" lower="0.0" upper="${finger_open_max}" />
     </joint>

File: toy_robot_ws/src/toy_robot_description/urdf/toy_robot.urdf.xacro (robot description, xacro)
@@ -7,3 +7,4 @@
     <xacro:include filename="$(find toy_robot_description)/urdf/arm_6dof.xacro" />
     <xacro:include filename="$(find toy_robot_description)/urdf/gripper.xacro" />
+    <xacro:include filename="$(find toy_robot_description)/urdf/gazebo_plugins.xacro" />
 </robot>
