Commit message: feat(description): add 2D LiDAR sensor for Nav2 support
- Add lidar.xacro: sensor link mounted on top of base
- Add LiDAR properties (radius, height, mass) to dimensions.xacro
- Add GPU LiDAR plugin to gazebo_plugins.xacro
  360-degree scan, 0.08-10.0m range, 10Hz update rate
- Add /scan bridge mapping to gz_bridge.yaml and gazebo.launch.xml
- Remove problematic colons from XML comments (YAML parse issue)
- Update URDF documentation with LiDAR inclusion order

Validated: /scan topic publishes LaserScan messages

File: toy_robot_ws/src/toy_robot_description/urdf/dimensions.xacro (robot description, xacro)
@@ -46,4 +46,8 @@
     <xacro:property name="finger_y_offset" value="0.02" />
     <xacro:property name="finger_open_max" value="0.025" />
+    <!-- LiDAR -->
+    <xacro:property name="lidar_radius" value="0.05" />
+    <xacro:property name="lidar_size_z" value="0.07" />
+    <xacro:property name="lidar_mass" value="0.27" />
     <!-- Wheels -->
     <xacro:property name="wheel_radius" value="0.05" />
@@ -61,4 +65,6 @@
     <!-- camera: near white -->
     <xacro:property name="color_camera" value="0.88 0.88 0.88 1.0" />
+    <!-- lidar: dark gray -->
+    <xacro:property name="color_lidar" value="0.25 0.25 0.25 1.0" />
     <!-- rubber dark -->
     <xacro:property name="color_wheel" value="0.15 0.15 0.15 1.0" />

File: toy_robot_ws/src/toy_robot_description/urdf/gazebo_plugins.xacro (robot description, xacro)
@@ -1,8 +1,6 @@
 <?xml version="1.0"?>
 <robot name="toy_robot" xmlns:xacro="http://www.ros.org/wiki/xacro">
-    <!-- =====================================================================
-         Gazebo material tags
-         Gazebo ignores URDF <material> tags and needs its own per-link entries.
-         ===================================================================== -->
+    <!-- Gazebo material tags -->
+    <!-- Gazebo ignores URDF material tags and needs its own per-link entries -->
     <gazebo reference="base_link">
         <visual>
@@ -131,17 +129,7 @@
         </visual>
     </gazebo>
-    <!-- Joint state publisher - broadcasts all joint positions so robot_state_publisher
-         can compute the full TF tree (arm, gripper) in both RViz and ROS. -->
-    <gazebo>
-        <plugin filename="gz-sim-joint-state-publisher-system"
-            name="gz::sim::systems::JointStatePublisher">
-            <topic>/joint_states</topic>
-        </plugin>
-    </gazebo>
-    <!-- =====================================================================
-         Differential drive plugin
-         Publishes /odom and subscribes to /cmd_vel.
-         wheel_separation = 2 * wheel_y = 2 * (base_radius + wheel_width/2)
-         ===================================================================== -->
+    <!-- Differential drive plugin for mobile base -->
+    <!-- Publishes /odom and subscribes to /cmd_vel -->
+    <!-- wheel_separation = 2 * wheel_y = 2 * (base_radius + wheel_width/2) -->
     <gazebo>
         <plugin filename="gz-sim-diff-drive-system"
@@ -163,10 +151,50 @@
         </plugin>
     </gazebo>
-    <!-- =====================================================================
-         Camera sensor
-         Publishes to /camera/image_raw (bridged via ros_gz_bridge).
-         The gz-sim-sensors-system must be loaded at world level in the launch
-         file for this sensor to activate.
-         ===================================================================== -->
+    <!-- Joint state publisher - broadcasts all joint positions -->
+    <!-- Allows robot_state_publisher to compute full TF tree -->
+    <!-- (arm, gripper) in both RViz and ROS nodes -->
+    <gazebo>
+        <plugin filename="gz-sim-joint-state-publisher-system"
+            name="gz::sim::systems::JointStatePublisher">
+            <topic>/joint_states</topic>
+        </plugin>
+    </gazebo>
+    <!-- 2D LiDAR sensor for Nav2 navigation -->
+    <!-- Mounted on top center of robot -->
+    <!-- Publishes to /scan (bridged via ros_gz_bridge) -->
+    <!-- Requires gz-sim-sensors-system loaded at world level -->
+    <gazebo reference="lidar_link">
+        <sensor name="lidar_sensor" type="gpu_lidar">
+            <pose>0 0 0 0 0 0</pose>
+            <lidar>
+                <scan>
+                    <horizontal>
+                        <samples>360</samples>
+                        <resolution>1</resolution>
+                        <min_angle>0</min_angle>
+                        <max_angle>6.28318</max_angle>
+                    </horizontal>
+                </scan>
+                <range>
+                    <min>0.08</min>
+                    <max>10.0</max>
+                    <resolution>0.01</resolution>
+                </range>
+                <noise>
+                    <type>gaussian</type>
+                    <mean>0</mean>
+                    <stddev>0.01</stddev>
+                </noise>
+            </lidar>
+            <always_on>true</always_on>
+            <update_rate>10</update_rate>
+            <visualize>false</visualize>
+            <topic>/scan</topic>
+        </sensor>
+    </gazebo>
+    <!-- Camera sensor RGB image -->
+    <!-- Mounted on front of robot -->
+    <!-- Publishes to /camera/image_raw (bridged via ros_gz_bridge) -->
+    <!-- Requires gz-sim-sensors-system loaded at world level -->
     <gazebo reference="camera_link">
         <sensor name="camera_sensor" type="camera">

File: toy_robot_ws/src/toy_robot_description/urdf/toy_robot.urdf.xacro (robot description, xacro)
@@ -5,4 +5,5 @@
     <xacro:include filename="$(find toy_robot_description)/urdf/wheels.xacro" />
     <xacro:include filename="$(find toy_robot_description)/urdf/camera.xacro" />
+    <xacro:include filename="$(find toy_robot_description)/urdf/lidar.xacro" />
     <xacro:include filename="$(find toy_robot_description)/urdf/arm_6dof.xacro" />
     <xacro:include filename="$(find toy_robot_description)/urdf/gripper.xacro" />

Commit message: fix(description): refine lidar mounting and inertia - Seat lidar flush on top of base_link - Keep compact lidar and camera visual dimensions - Correct cylinder inertia formula for lidar (ixx/iyy)

File: toy_robot_ws/src/toy_robot_description/urdf/dimensions.xacro (robot description, xacro)
@@ -6,8 +6,8 @@
     <xacro:property name="base_mass" value="2.0" />
     <!-- Camera -->
-    <xacro:property name="camera_size_x" value="0.04" />
-    <xacro:property name="camera_size_y" value="0.08" />
-    <xacro:property name="camera_size_z" value="0.03" />
-    <xacro:property name="camera_mass" value="0.1" />
+    <xacro:property name="camera_size_x" value="0.03" />
+    <xacro:property name="camera_size_y" value="0.05" />
+    <xacro:property name="camera_size_z" value="0.022" />
+    <xacro:property name="camera_mass" value="0.07" />
     <xacro:property name="camera_mount_x" value="${base_radius}" />
     <xacro:property name="camera_mount_z" value="${base_height/2}" />
@@ -47,7 +47,7 @@
     <xacro:property name="finger_open_max" value="0.025" />
     <!-- LiDAR -->
-    <xacro:property name="lidar_radius" value="0.05" />
-    <xacro:property name="lidar_size_z" value="0.07" />
-    <xacro:property name="lidar_mass" value="0.27" />
+    <xacro:property name="lidar_radius" value="0.032" />
+    <xacro:property name="lidar_size_z" value="0.038" />
+    <xacro:property name="lidar_mass" value="0.16" />
     <!-- Wheels -->
     <xacro:property name="wheel_radius" value="0.05" />

File: toy_robot_ws/src/toy_robot_description/urdf/lidar.xacro (robot description, xacro)
@@ -8,5 +8,5 @@
         <parent link="base_link" />
         <child link="lidar_link" />
-        <origin xyz="0 0 ${base_height/2 + lidar_size_z/2}" rpy="0 0 0" />
+        <origin xyz="0 0 ${base_height + lidar_size_z/2}" rpy="0 0 0" />
     </joint>
     <!-- LiDAR link -->
@@ -31,8 +31,8 @@
             <mass value="${lidar_mass}" />
             <inertia
-                ixx="${lidar_mass * (lidar_radius * lidar_radius + lidar_size_z * lidar_size_z) / 12}"
+                ixx="${lidar_mass * (3 * lidar_radius * lidar_radius + lidar_size_z * lidar_size_z) / 12}"
                 ixy="0"
                 ixz="0"
-                iyy="${lidar_mass * (lidar_radius * lidar_radius + lidar_size_z * lidar_size_z) / 12}"
+                iyy="${lidar_mass * (3 * lidar_radius * lidar_radius + lidar_size_z * lidar_size_z) / 12}"
                 iyz="0"
                 izz="${lidar_mass * lidar_radius * lidar_radius / 2}" />
