Commit message: tune(sim): improve base stability and lidar integration
- seat lidar flush on base top and correct lidar inertia formula
- compact camera/lidar visual dimensions
- increase base mass and lower lidar mass for better pitch stability
- lower diff-drive acceleration limits to reduce forward tilt during teleop

File: toy_robot_ws/src/toy_robot_description/urdf/base_mobile.xacro (robot description, xacro)
@@ -24,5 +24,5 @@
         </collision>
         <inertial>
-            <origin xyz="0 0 ${base_height/2}" rpy="0 0 0" />
+            <origin xyz="0 0 ${base_height * 0.4}" rpy="0 0 0" />
             <mass value="${base_mass}" />
             <inertia

File: toy_robot_ws/src/toy_robot_description/urdf/dimensions.xacro (robot description, xacro)
@@ -4,5 +4,5 @@
     <xacro:property name="base_radius" value="0.2" />
     <xacro:property name="base_height" value="0.1" />
-    <xacro:property name="base_mass" value="2.0" />
+    <xacro:property name="base_mass" value="3.5" />
     <!-- Camera -->
     <xacro:property name="camera_size_x" value="0.03" />
@@ -49,5 +49,5 @@
     <xacro:property name="lidar_radius" value="0.032" />
     <xacro:property name="lidar_size_z" value="0.038" />
-    <xacro:property name="lidar_mass" value="0.16" />
+    <xacro:property name="lidar_mass" value="0.08" />
     <!-- Wheels -->
     <xacro:property name="wheel_radius" value="0.05" />

File: toy_robot_ws/src/toy_robot_description/urdf/gazebo_plugins.xacro (robot description, xacro)
@@ -139,8 +139,8 @@
             <wheel_separation>${2 * wheel_y}</wheel_separation>
             <wheel_radius>${wheel_radius}</wheel_radius>
-            <max_linear_acceleration>1.0</max_linear_acceleration>
-            <min_linear_acceleration>-1.0</min_linear_acceleration>
-            <max_angular_acceleration>2.0</max_angular_acceleration>
-            <min_angular_acceleration>-2.0</min_angular_acceleration>
+            <max_linear_acceleration>0.25</max_linear_acceleration>
+            <min_linear_acceleration>-0.25</min_linear_acceleration>
+            <max_angular_acceleration>0.9</max_angular_acceleration>
+            <min_angular_acceleration>-0.9</min_angular_acceleration>
             <odom_publish_frequency>20</odom_publish_frequency>
             <topic>/cmd_vel</topic>
