Commit message: Add differential drive robot simulation milestone

File: projects/differential_drive_ws/src/differential_drive_robot/urdf/differential_drive_robot.urdf.xacro (robot description, xacro)
@@ -5,30 +5,4 @@
     <xacro:include filename="$(find differential_drive_robot)/urdf/base.xacro" />
     <xacro:include filename="$(find differential_drive_robot)/urdf/wheels.xacro" />
-    <link name="caster_link">
-        <visual>
-            <origin xyz="0 0 0" rpy="0 0 0" />
-            <geometry>
-                <sphere radius="${caster_radius}" />
-            </geometry>
-            <material name="gray" />
-        </visual>
-        <collision>
-            <origin xyz="0 0 0" rpy="0 0 0" />
-            <geometry>
-                <sphere radius="${caster_radius}" />
-            </geometry>
-        </collision>
-        <inertial>
-            <origin xyz="0 0 0" rpy="0 0 0" />
-            <mass value="${caster_mass}" />
-            <inertia ixx="${caster_inertia_ixx}" ixy="0.0" ixz="0.0"
-                iyy="${caster_inertia_iyy}" iyz="0.0"
-                izz="${caster_inertia_izz}" />
-        </inertial>
-    </link>
-    <joint name="caster_joint" type="fixed">
-        <parent link="base_link" />
-        <child link="caster_link" />
-        <origin xyz="0.12 0 -0.03" rpy="0 0 0" />
-    </joint>
+    <xacro:include filename="$(find differential_drive_robot)/urdf/gazebo_plugins.xacro" />
 </robot>

File: projects/differential_drive_ws/src/differential_drive_robot/urdf/materials.xacro (robot description, xacro)
@@ -1,9 +1,11 @@
 <?xml version="1.0"?>
 <robot xmlns:xacro="http://wiki.ros.org/xacro">
+    <xacro:property name="color_base" value="0.2 0.4 0.8 1.0" />
+    <xacro:property name="color_wheel" value="0.1 0.1 0.1 1.0" />
     <material name="blue">
-        <color rgba="0.2 0.4 0.8 1.0" />
+        <color rgba="${color_base}" />
     </material>
     <material name="black">
-        <color rgba="0.1 0.1 0.1 1.0" />
+        <color rgba="${color_wheel}" />
     </material>
     <material name="gray">

File: projects/differential_drive_ws/src/differential_drive_robot/urdf/wheels.xacro (robot description, xacro)
@@ -57,3 +57,30 @@
         <axis xyz="0 1 0" />
     </joint>
+    <link name="caster_link">
+        <visual>
+            <origin xyz="0 0 0" rpy="0 0 0" />
+            <geometry>
+                <sphere radius="${caster_radius}" />
+            </geometry>
+            <material name="gray" />
+        </visual>
+        <collision>
+            <origin xyz="0 0 0" rpy="0 0 0" />
+            <geometry>
+                <sphere radius="${caster_radius}" />
+            </geometry>
+        </collision>
+        <inertial>
+            <origin xyz="0 0 0" rpy="0 0 0" />
+            <mass value="${caster_mass}" />
+            <inertia ixx="${caster_inertia_ixx}" ixy="0.0" ixz="0.0"
+                iyy="${caster_inertia_iyy}" iyz="0.0"
+                izz="${caster_inertia_izz}" />
+        </inertial>
+    </link>
+    <joint name="caster_joint" type="fixed">
+        <parent link="base_link" />
+        <child link="caster_link" />
+        <origin xyz="0.12 0 -0.03" rpy="0 0 0" />
+    </joint>
 </robot>
